File: Keypad_Board.kicad_pcb (KiCad board)
At the start: 2 copper layers, 45 x 61 mm, 40 parts, among them IC1 STM32L010K4T6, IC2 TMUX136RSER, J3 Data_Conn, J4 SEL Jumper, J5 SW_Header, J6 BOOT Jumper

Commit message: update
Parts:
- moved H1 1.00 mm to (114.5, 53.5)
- moved H2 1.00 mm to (150.5, 53.5)
- moved J3 0.93 mm to (130.5, 53.2)
Connections:
- J5 pad 3: /SYS_SWDIO -> /NRST
- J5 pad 4: /SYS_SWCLK -> /SYS_SWDIO
- J5 pad 5: /NRST -> /SYS_SWCLK
Routing:
- net +3.3V: track 18.6 -> 38.5 mm
- net /I2C1_SCL: track 0.00 -> 9.80 mm
- net /I2C1_SDA: track 0.00 -> 9.53 mm
- net /PA8: track 24.0 -> 20.0 mm
- net /SYS_SWDIO: track 7.90 -> 6.32 mm
- net /PA11: track 53.5 -> 54.5 mm
- net /PA10: track 42.6 -> 43.6 mm
- net /SYS_SWCLK: track 6.65 -> 6.05 mm
- net /PB1: track 37.9 -> 38.1 mm, vias 0 -> 2
- net /PA5: track 41.3 -> 41.4 mm, vias 0 -> 2
- net GND: vias 10 -> 21
Other:
- board size 45 x 61 mm -> 45 x 62 mm
- board text added: "3"
- board text added: "4"
- board text added: "5"
- board text added: "6"
- board text added: "I2C/LPUART"
- board text added: "UPD/STR"

Commit message: Update
Parts:
- moved C14 8.96 mm to (129.9, 56.1)
- moved IC2 8.80 mm to (134.2, 57.0)
- moved C12 5.48 mm to (119.0, 59.1), turned to 180 degrees
- moved C11 3.89 mm to (122.9, 66.8), turned to -90 degrees
- moved C9 2.89 mm to (122.9, 61.5), turned to 90 degrees
- moved C10 2.45 mm to (138.8, 69.2)
- moved IC1 2.21 mm to (132.4, 65.4)
- moved J3 1.20 mm to (129.3, 53.1)
- moved U9 1.18 mm to (120.5, 66.0)
- moved J6 1.14 mm to (114.8, 59.7)
- moved J5 0.61 mm to (144.4, 70.2)
- moved J4 0.50 mm to (125.5, 53.1)
Connections:
- J5 pad 3: /NRST -> /SYS_SWDIO
- J5 pad 4: /SYS_SWDIO -> /SYS_SWCLK
- J5 pad 5: /SYS_SWCLK -> /NRST
Routing:
- net /PA11: track 54.5 -> 12.3 mm
- net /NRST: track 11.8 -> 42.0 mm, vias 0 -> 4
- net +3.3V: track 38.5 -> 63.6 mm, vias 0 -> 5
- net /PA10: track 43.6 -> 22.3 mm, vias 2 -> 1
- net /PA9: track 31.7 -> 13.7 mm, vias 2 -> 1
- net /PA8: track 20.0 -> 6.58 mm, vias 2 -> 1
- net /SEL: track 3.79 -> 16.8 mm, vias 0 -> 1
- net /COM2: track 15.2 -> 4.24 mm
- net /COM1: track 13.1 -> 3.39 mm
- net /LPUART1_TX: track 27.5 -> 18.3 mm, vias 2 -> 0
- net /LPUART1_RX: track 25.9 -> 17.2 mm, vias 2 -> 0
- net /I2C1_SCL: track 9.80 -> 5.11 mm
- net /I2C1_SDA: track 9.53 -> 5.39 mm
- net /PA2: track 17.0 -> 14.5 mm
- net /SYS_SWCLK: track 6.05 -> 8.28 mm
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Other:
- board text removed: "I2C/LPUART"
- board text removed: "UPD/STR"

Commit message: Update
Parts:
- moved C10 0.59 mm to (138.8, 69.7)
Routing:
- net /PA11: track 12.3 -> 54.6 mm, vias 2 -> 4
- net +3.3V: track 63.6 -> 101.9 mm, vias 5 -> 7
- net /PA10: track 22.3 -> 42.9 mm, vias 1 -> 2
- net /PA9: track 13.7 -> 32.2 mm, vias 1 -> 2
- net /PA8: track 6.58 -> 21.8 mm, vias 1 -> 0
- net /BOOT0: track 23.4 -> 22.5 mm
- net GND: vias 35 -> 56
Other:
- board text added: "I2C/LPUART"
- board text added: "STM32L010K4T6 MCU Based I2C/LPUART Keypad"
- board text added: "UPD/STR"

Commit message: Update
Connections:
- IC1 pad 25: unconnected-(IC1-PA15-Pad25) -> /SEL
Routing:
- net /SEL: track 16.8 -> 42.6 mm, vias 1 -> 4
- net GND: vias 56 -> 60
Other:
- board text added: "0"
- board text added: "7"
- board text added: "8"
- board text added: "9"

Commit message: Update
Parts:
- moved C12 33.5 mm to (90.2, 41.8)
- moved C13 33.5 mm to (93.7, 58.8)
- moved C14 33.5 mm to (101.2, 38.9)
- moved C15 33.5 mm to (93.7, 66.8)
- moved C16 33.5 mm to (93.7, 74.8)
- moved C17 33.5 mm to (93.7, 82.8)
- moved C18 33.5 mm to (106.7, 58.8)
- moved C19 33.5 mm to (106.7, 66.8)
- moved C20 33.5 mm to (106.7, 74.8)
- moved C21 33.5 mm to (106.7, 82.8)
- moved C22 33.5 mm to (119.7, 58.8)
- moved C23 33.5 mm to (119.7, 66.8)
- moved C24 33.5 mm to (119.7, 74.8)
- moved U14 33.5 mm to (99.8, 60.4)
- moved U15 33.5 mm to (99.8, 68.4)
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