File: Keypad_Board.kicad_pcb (KiCad board)
At the start: 2 copper layers, 45 x 62 mm, 40 parts, among them IC1 STM32L010K4T6, IC2 TMUX136RSER, J3 Data_Conn, J4 SEL Jumper, J5 SW_Header, J6 BOOT Jumper

Commit message: Update
Routing:
- net +3.3V: track 101.9 -> 116.7 mm, vias 7 -> 9
- net GND: vias 60 -> 64
Changed lines of the file:
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@@
+	)
+	(via
+		(at 106.73 61.16)
+		(size 0.7)
+		(drill 0.3)
+		(layers "F.Cu" "B.Cu")
+		(free yes)
+		(net 1)
 	)
 	(via
@@
 	)
 	(via
+		(at 98.72 61.15)
+		(size 0.7)
+		(drill 0.3)
+		(layers "F.Cu" "B.Cu")
+		(free yes)
+		(net 1)
+	)
+	(via
+		(at 92.26 62.91)
+		(size 0.7)
+		(drill 0.3)
+		(layers "F.Cu" "B.Cu")
+		(free yes)
+		(net 1)
+	)
+	(via
 		(at 91.21 45.91)
 		(size 0.7)
@@
 	)
 	(via
-		(at 106.66 61.44)
+		(at 106.75 63.12)
 		(size 0.7)
 		(drill 0.3)
@@
 	)
 	(via
-		(at 111.4 56.12)
+		(at 112.41 54.41)
 		(size 0.7)
 		(drill 0.3)
@@
 	)
 	(via
+		(at 99.29 62.99)
+		(size 0.7)
+		(drill 0.3)
+		(layers "F.Cu" "B.Cu")
+		(free yes)
+		(net 1)
+	)
+	(via
 		(at 105.27 80.11)
 		(size 0.7)
@@
 	)
 	(via
-		(at 112.42 54.83)
+		(at 110.25 55.08)
 		(size 0.7)
 		(drill 0.3)
@@
 	)
 	(via
-		(at 93.68 61.35)
+		(at 93.8 61.34)
 		(size 0.7)
 		(drill 0.3)
@@
 	)
 	(segment
-		(start 87.59 54.96)
-		(end 84.92 52.29)
-		(width 0.25)
-		(layer "F.Cu")
-		(net 2)
-	)
-	(segment
 		(start 86.89 40.27)
 		(end 87.84 40.27)
@@
 	)
 	(segment
-		(start 92.19 54.96)
-		(end 87.59 54.96)
-		(width 0.25)
-		(layer "F.Cu")
-		(net 2)
-	)
-	(segment
 		(start 87.84 40.27)
 		(end 89.54 38.57)
@@
 	)
 	(segment
+		(start 99.3 62.08)
+		(end 99.26 62.04)
+		(width 0.25)
+		(layer "F.Cu")
+		(net 2)
+	)
+	(segment
 		(start 83.8 51.17)
 		(end 84.92 52.29)
@@
 	)
 	(segment
+		(start 106.76 62.08)
+		(end 99.3 62.08)
+		(width 0.25)
+		(layer "F.Cu")
+		(net 2)
+	)
+	(segment
 		(start 107.93 50.97)
 		(end 109.5475 50.97)
@@
 	)
 	(segment
+		(start 84.92 60.34)
+		(end 84.92 52.29)
+		(width 0.25)
+		(layer "F.Cu")
+		(net 2)
+	)
+	(segment
 		(start 97.95 45.37)
 		(end 97.92 45.34)
@@
 	)
 	(segment
+		(start 92.83 62.04)
+		(end 86.62 62.04)
+		(width 0.25)
+		(layer "F.Cu")
+		(net 2)
+	)
+	(segment
 		(start 94.17 48.5525)
 		(end 94.15 48.5725)
@@
 	)
 	(segment
+		(start 86.62 62.04)
+		(end 84.92 60.34)
+		(width 0.25)
+		(layer "F.Cu")
+		(net 2)
+	)
+	(segment
 		(start 83.8 51.06)
 		(end 83.8 51.17)
@@
 	)
 	(via
+		(at 99.26 62.04)
+		(size 0.7)
+		(drill 0.3)
+		(layers "F.Cu" "B.Cu")
+		(net 2)
+	)
+	(via
 		(at 95.94 45.34)
 		(size 0.7)
@@
 	)
 	(via
-		(at 92.19 54.96)
-		(size 0.7)
-		(drill 0.3)
-		(layers "F.Cu" "B.Cu")
-		(net 2)
-	)
-	(via
 		(at 97.95 48.55)
 		(size 0.7)
@@
 	)
 	(via
+		(at 106.76 62.08)
+		(size 0.7)
+		(drill 0.3)
+		(layers "F.Cu" "B.Cu")
+		(net 2)
+	)
+	(via
 		(at 83.8 51.06)
+		(size 0.7)
+		(drill 0.3)
+		(layers "F.Cu" "B.Cu")
+		(net 2)
+	)
+	(via
+		(at 92.83 62.04)
 		(size 0.7)
 		(drill 0.3)
@@
 	)
 	(segment
+		(start 99.26 62.04)
+		(end 92.83 62.04)
+		(width 0.25)
+		(layer "B.Cu")
+		(net 2)
+	)
+	(segment
+		(start 112.64 52.98)
+		(end 111.72 53.9)
+		(width 0.25)
+		(layer "B.Cu")
+		(net 2)
+	)
+	(segment
 		(start 84.545 42.445)
 		(end 83.84 43.15)
@@
 	)
 	(segment
-		(start 112.64 52.98)
-		(end 110.66 54.96)
+		(start 106.775 62.065)
+		(end 106.76 62.08)
+		(width 0.25)
+		(layer "B.Cu")
+		(net 2)
+	)
+	(segment
+		(start 110.665 62.065)
+		(end 107.565 62.065)
 		(width 0.25)
 		(layer "B.Cu")
@@
 	)
 	(segment
-		(start 110.66 54.96)
-		(end 92.19 54.96)
+		(start 107.565 62.065)
+		(end 106.775 62.065)
 		(width 0.25)
 		(layer "B.Cu")
@@
 		(width 0.25)
 		(layer "B.Cu")
+		(net 2)
+	)
+	(segment
+		(start 111.72 53.9)
+		(end 111.72 61.01)
+		(width 0.25)
+		(layer "B.Cu")
+		(net 2)
+	)
+	(segment
+		(start 111.72 61.01)
+		(end 110.665 62.065)
+		(width 0.25)
+		(layer "B.Cu")
