File: Keypad_Board.kicad_pcb (KiCad board)
At the start: 2 copper layers, 45 x 62 mm, 40 parts, among them IC1 STM32L010K4T6, IC2 TMUX136RSER, J3 Data_Conn, J4 SEL Jumper, J5 SW_Header, J6 BOOT Jumper

Commit message: Update
Parts:
- added J1: Data_Conn_Header, Connector_PinHeader_2.54mm:PinHeader_1x04_P2.54mm_Vertical, F.Cu at (100.5, 40.2)
- added J2: Pin_Header, Connector_PinHeader_2.54mm:PinHeader_1x04_P2.54mm_Vertical, F.Cu at (118.0, 42.9)
- added R1: 100R, Resistor_SMD:R_0805_2012Metric_Pad1.20x1.40mm_HandSolder, F.Cu at (91.5, 52.4)
- added R2: 100R, Resistor_SMD:R_0805_2012Metric_Pad1.20x1.40mm_HandSolder, F.Cu at (89.4, 52.4)
- added R3: 100R, Resistor_SMD:R_0805_2012Metric_Pad1.20x1.40mm_HandSolder, F.Cu at (134.9, 56.9)
- added R4: 100R, Resistor_SMD:R_0805_2012Metric_Pad1.20x1.40mm_HandSolder, F.Cu at (134.9, 59.8)
- C10, C11, C12, C13, C14, C15, C16, C17, C18, C19, C20, C21, C22, C23, C24, C25, C9: footprint Capacitor_SMD:C_0805_2012Metric_Pad1.18x1.45mm_HandSolder -> Capacitor_SMD:C_0603_1608Metric_Pad1.08x0.95mm_HandSolder
- J3: value Data_Conn -> Data_Conn_Socket; footprint Connector_PinHeader_2.54mm:PinHeader_1x04_P2.54mm_Horizontal -> Connector_PinSocket_2.54mm:PinSocket_1x04_P2.54mm_Vertical; moved to B.Cu
- J5: footprint Connector_PinSocket_2.54mm:PinSocket_1x05_P2.54mm_Horizontal -> Connector_PinHeader_2.54mm:PinHeader_1x05_P2.54mm_Vertical
- moved C12 9.43 mm to (86.1, 50.3)
- moved U9 9.43 mm to (87.7, 57.2)
- moved C9 7.76 mm to (95.7, 51.9), turned to 180 degrees
- moved C14 6.60 mm to (101.2, 45.5)
- moved IC1 6.60 mm to (103.7, 54.8)
- moved IC2 6.60 mm to (105.5, 46.4)
- moved U10 6.60 mm to (86.8, 67.0)
- moved U14 6.60 mm to (99.8, 67.0)
- moved U18 6.60 mm to (112.8, 67.0)
- moved C10 6.60 mm to (110.1, 59.1)
- moved C13 6.60 mm to (93.7, 65.4)
- moved C18 6.60 mm to (106.7, 65.4)
- moved C22 6.60 mm to (119.7, 65.4)
- moved J5 5.87 mm to (121.6, 52.8)
- moved C11 5.51 mm to (95.7, 54.9), turned to 180 degrees
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Connections:
- IC1 pad 22: unconnected-(IC1-PA12-Pad22) -> /PA12
- IC1 pad 26: unconnected-(IC1-PB3-Pad26) -> /PB3
- IC1 pad 27: unconnected-(IC1-PB4-Pad27) -> /PB4
- IC1 pad 28: unconnected-(IC1-PB5-Pad28) -> /PB5
- IC2 pad 1: /LPUART1_TX -> Net-(IC2-A1)
- IC2 pad 2: /LPUART1_RX -> Net-(IC2-A2)
- IC2 pad 3: /I2C1_SDA -> Net-(IC2-B1)
- IC2 pad 4: /I2C1_SCL -> Net-(IC2-B2)
Routing:
- net /PA11: track 54.6 -> 32.1 mm
- net +3.3V: track 116.7 -> 97.4 mm, vias 9 -> 5
- net /PA10: track 42.9 -> 24.7 mm
- net /PA9: track 32.2 -> 17.8 mm
- net /BOOT0: track 22.5 -> 14.5 mm
- net /LPUART1_TX: track 18.3 -> 10.9 mm, vias 0 -> 1
- net /LPUART1_RX: track 17.2 -> 10.1 mm, vias 0 -> 1
- net Net-(IC2-A2): track 0.00 -> 6.78 mm
- net Net-(IC2-A1): track 0.00 -> 6.17 mm
- net /NRST: track 42.0 -> 36.1 mm, vias 4 -> 3
- net /PB1: track 37.8 -> 33.3 mm
- net /PA5: track 39.2 -> 34.7 mm
- net GND: track 8.49 -> 12.3 mm, vias 64 -> 46
- net /COM2: track 4.24 -> 0.79 mm
- net /PB0: track 29.2 -> 26.2 mm
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Other:
- board size 45 x 62 mm -> 45 x 64 mm
- board text added: "3V/GN/DI/CL/NR"
- board text added: "NRST"
- board text added: "SPI1"

Commit message: Update
Parts:
- moved R4 40.7 mm to (96.2, 47.3), turned to 180 degrees
- moved R3 39.4 mm to (96.2, 49.5), turned to 180 degrees
- moved IC2 13.6 mm to (92.0, 45.4)
- moved C14 12.4 mm to (88.8, 44.6), turned to 90 degrees
- moved R1 2.46 mm to (89.3, 53.5)
- moved R2 2.37 mm to (91.5, 53.5)
- moved J2 2.12 mm to (115.9, 42.6)
- moved J1 0.10 mm to (100.6, 40.2)
Connections:
- IC1 pad 25: /SEL -> /PA15
- IC1 pad 28: /PB5 -> /SEL
- J2 pad 1: /PB5 -> /PB4
- J2 pad 2: /PB4 -> /PB3
- J2 pad 3: /PB3 -> /PA15
Routing:
- net +3.3V: track 97.4 -> 128.9 mm
- net /NRST: track 36.1 -> 60.6 mm, vias 3 -> 5
- net /COM2: track 0.79 -> 21.3 mm, vias 0 -> 1
- net /COM1: track 0.90 -> 19.1 mm, vias 0 -> 1
- net /PB4: track 0.00 -> 16.1 mm
- net /PA11: track 32.1 -> 46.8 mm, vias 4 -> 2
- net /PA10: track 24.7 -> 38.1 mm, vias 2 -> 0
- net /SYS_SWDIO: track 6.07 -> 19.4 mm, vias 0 -> 1
- net /PB3: track 0.00 -> 13.0 mm
- net /SYS_SWCLK: track 7.40 -> 19.9 mm, vias 0 -> 1
- net /SEL: track 41.5 -> 53.8 mm, vias 3 -> 2
- net /PA9: track 17.8 -> 29.3 mm, vias 2 -> 0
- net /PA12: track 0.00 -> 10.9 mm, vias 0 -> 1
- net /PA15: track 0.00 -> 10.6 mm
- net /BOOT0: track 14.5 -> 20.4 mm
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Other:
- board text added: "A12/B3/B4/B5"
- board text added: "CL/DA/GN/3V"
- board text added: "RX/TX/GN/3V"

Commit message: Update
Parts:
- added FB1: BLM21PG601SN1D_0805, Capacitor_SMD:C_0805_2012Metric_Pad1.18x1.45mm_HandSolder, F.Cu at (130.4, 47.6)
Connections:
- C11 pad 1: +3.3V -> /VDDA
- IC1 pad 5: +3.3V -> /VDDA
Changed lines of the file:
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@@
 	(net 33 "Net-(IC2-A1)")
 	(net 34 "/PA15")
+	(net 35 "/VDDA")
 	(footprint "Personal_Project:Button_KMR231GLFS"
 		(layer "F.Cu")
@@
 			(layers "F.Cu" "F.Paste" "F.Mask")
 			(roundrect_rratio 0.25)
-			(net 2 "+3.3V")
+			(net 35 "/VDDA")
 			(pintype "passive")
 		)
@@
 		)
 	)
+	(footprint "Capacitor_SMD:C_0805_2012Metric_Pad1.18x1.45mm_HandSolder"
+		(layer "F.Cu")
+		(at 130.4225 47.64)
+		(descr "Capacitor SMD 0805 (2012 Metric), square (rectangular) end terminal, IPC_7351 nominal with elongated pad for handsoldering. (Body size source: IPC-SM-782 page 76, https://www.pcb-3d.com/wordpress/wp-content/uploads/ipc-sm-782a_amendment_1_and_2.pdf, https://docs.google.com/spreadsheets/d/1BsfQQcO9C6DZCsRaXUlFlo91Tg2WpOkGARC1WS5S8t0/edit?usp=sharing), generated with kicad-footprint-generator")
+		(tags "capacitor handsolder")
+		(property "Reference" "FB1"
+			(at 0 -1.68 0)
+			(layer "F.SilkS")
+			(effects
+				(font
+					(size 1 1)
+					(thickness 0.15)
+				)
+			)
+		)
+		(property "Value" "BLM21PG601SN1D_0805"
+			(at 0 1.68 0)
+			(layer "F.Fab")
+			(effects
+				(font
+					(size 1 1)
+					(thickness 0.15)
+				)
+			)
+		)
+		(property "Footprint" "Capacitor_SMD:C_0805_2012Metric_Pad1.18x1.45mm_HandSolder"
+			(at 0 0 0)
+			(unlocked yes)
+			(layer "F.Fab")
+			(hide yes)
+			(effects
+				(font
+					(size 1.27 1.27)
+					(thickness 0.15)
+				)
+			)
+		)
+		(property "Datasheet" ""
+			(at 0 0 0)
+			(unlocked yes)
+			(layer "F.Fab")
+			(hide yes)
+			(effects
+				(font
+					(size 1.27 1.27)
+					(thickness 0.15)
+				)
+			)
+		)
+		(property "Description" "Ferrite bead"
+			(at 0 0 0)
+			(unlocked yes)
+			(layer "F.Fab")
+			(hide yes)
+			(effects
+				(font
+					(size 1.27 1.27)
+					(thickness 0.15)
+				)
+			)
+		)
+		(property ki_fp_filters "Inductor_* L_* *Ferrite*")
+		(sheetname "Root")
+		(sheetfile "Keypad_Board.kicad_sch")
+		(attr smd)
+		(fp_line
+			(start -0.261252 -0.735)
+			(end 0.261252 -0.735)
+			(stroke
+				(width 0.12)
+				(type solid)
+			)
+			(layer "F.SilkS")
+		)
+		(fp_line
+			(start -0.261252 0.735)
+			(end 0.261252 0.735)
+			(stroke
+				(width 0.12)
+				(type solid)
+			)
+			(layer "F.SilkS")
+		)
+		(fp_line
+			(start -1.88 -0.98)
+			(end 1.88 -0.98)
+			(stroke
+				(width 0.05)
+				(type solid)
+			)
+			(layer "F.CrtYd")
+		)
+		(fp_line
+			(start -1.88 0.98)
+			(end -1.88 -0.98)
+			(stroke
+				(width 0.05)
+				(type solid)
+			)
+			(layer "F.CrtYd")
+		)
+		(fp_line
+			(start 1.88 -0.98)
+			(end 1.88 0.98)
+			(stroke
+				(width 0.05)
+				(type solid)
+			)
+			(layer "F.CrtYd")
+		)
+		(fp_line
+			(start 1.88 0.98)
+			(end -1.88 0.98)
+			(stroke
+				(width 0.05)
+				(type solid)
+			)
+			(layer "F.CrtYd")
+		)
+		(fp_line
+			(start -1 -0.625)
+			(end 1 -0.625)
+			(stroke
+				(width 0.1)
+				(type solid)
+			)
+			(layer "F.Fab")
+		)
+		(fp_line
+			(start -1 0.625)
+			(end -1 -0.625)
+			(stroke
+				(width 0.1)
+				(type solid)
+			)
+			(layer "F.Fab")
+		)
+		(fp_line
+			(start 1 -0.625)
+			(end 1 0.625)
+			(stroke
+				(width 0.1)
+				(type solid)
+			)
+			(layer "F.Fab")
+		)
+		(fp_line
+			(start 1 0.625)
+			(end -1 0.625)
+			(stroke
+				(width 0.1)
+				(type solid)
+			)
+			(layer "F.Fab")
+		)
+		(fp_text user "${REFERENCE}"
+			(at 0 0 0)
+			(layer "F.Fab")
+			(effects
+				(font
+					(size 0.5 0.5)
+					(thickness 0.08)
+				)
+			)
+		)
+		(pad "1" smd roundrect
+			(at -1.0375 0)
+			(size 1.175 1.45)
+			(layers "F.Cu" "F.Paste" "F.Mask")
+			(roundrect_rratio 0.212766)
+			(net 2 "+3.3V")
+			(pintype "passive")
+		)
+		(pad "2" smd roundrect
+			(at 1.0375 0)
+			(size 1.175 1.45)
+			(layers "F.Cu" "F.Paste" "F.Mask")
+			(roundrect_rratio 0.212766)
+			(net 35 "/VDDA")
+			(pintype "passive")
+		)
+		(model "${KICAD8_3DMODEL_DIR}/Capacitor_SMD.3dshapes/C_0805_2012Metric.wrl"
+			(offset
+				(xyz 0 0 0)
+			)
+			(scale
+				(xyz 1 1 1)
+			)
+			(rotate
+				(xyz 0 0 0)
+			)
+		)
+	)
 	(footprint "Capacitor_SMD:C_0603_1608Metric_Pad1.08x0.95mm_HandSolder"
 		(layer "F.Cu")
@@
 			(size 0.6 1.475)
 			(layers "F.Cu" "F.Paste" "F.Mask")
-			(net 2 "+3.3V")
+			(net 35 "/VDDA")
 			(pinfunction "VDDA")
 			(pintype "passive")
@@
 		(tags "resistor handsolder")
 		(property "Reference" "R4"
-			(at 0 -1.65 360)
+			(at 0 -1.65 0)
 			(layer "F.SilkS")
 			(effects
@@
 		)
 		(property "Value" "100R"
-			(at 0 1.65 360)
+			(at 0 1.65 0)
 			(layer "F.Fab")
 			(effects
@@
 		)
 		(fp_text user "${REFERENCE}"
-			(at 0 0 360)
+			(at 0 0 0)
 			(layer "F.Fab")
 			(effects
@@
 		(tags "resistor handsolder")
 		(property "Reference" "R3"
-			(at 0 -1.65 360)
+			(at 0 -1.65 0)
 			(layer "F.SilkS")
 			(effects
@@
 		)
 		(property "Value" "100R"
-			(at 0 1.65 360)
+			(at 0 1.65 0)
 			(layer "F.Fab")
 			(effects
@@
 		)
 		(fp_text user "${REFERENCE}"
-			(at 0 0 360)
+			(at 0 0 0)
 			(layer "F.Fab")
 			(effects

Commit message: Update
Parts:
- removed FB1: BLM21PG601SN1D_0805, Capacitor_SMD:C_0805_2012Metric_Pad1.18x1.45mm_HandSolder
Connections:
- C11 pad 1: /VDDA -> +3.3V
- IC1 pad 5: /VDDA -> +3.3V
Routing:
- net /PA8: track 21.8 -> 19.7 mm
