File: Keypad_Board.kicad_sch (KiCad schematic)
At the start: 41 parts, among them J1 Conn_02x05_Odd_Even, J2 Button_Expansion_Connector, U9 STM32L010K4T6

Commit message: Update
Parts:
- removed C1, C2, C3, C4, C5, C6, C7, C8: 1u, Capacitor_SMD:C_0805_2012Metric_Pad1.18x1.45mm_HandSolder, symbol Device:C
- removed ESD1, ESD2: ESDALC6V1W5, Personal_Project:SOT323-5L_STM-L, symbol Personal_Projects:ESDALC6V1W5
- removed J1: Conn_02x05_Odd_Even, Connector_PinHeader_2.54mm:PinHeader_2x05_P2.54mm_Vertical, symbol Connector_Generic:Conn_02x05_Odd_Even
- removed J2: Button_Expansion_Connector, Personal_Project:WR-PHD 2.54 MM DUAL SOCKET HEADE, symbol Personal_Projects:WR-PHD 2.54 MM DUAL SOCKET HEADE
- removed R1, R11, R13, R15, R3, R5, R7, R9: 100k, Resistor_SMD:R_0805_2012Metric_Pad1.20x1.40mm_HandSolder, symbol Device:R
- removed R10, R12, R14, R16, R2, R4, R6, R8: 1k, Resistor_SMD:R_0805_2012Metric_Pad1.20x1.40mm_HandSolder, symbol Device:R
- removed U1, U2, U3, U4, U5, U6, U7, U8: ~, Personal_Project:Button_KMR231GLFS, symbol Personal_Projects:Button_KMR231GLFS
- removed U9: STM32L010K4T6, Package_QFP:LQFP-32_7x7mm_P0.8mm, symbol MCU_ST_STM32L0:STM32L010K4Tx
- added C10, C11, C12, C13, C14, C15, C16, C17, C18, C19, C20, C21, C22, C23, C24, C25, C9: 100n, Capacitor_SMD:C_0805_2012Metric_Pad1.18x1.45mm_HandSolder, symbol Device:C
- added IC1: STM32L010K4T6, Personal_Project:STM32L010K4T6 _QFP80P900X900X160-32N, symbol Personal_Projects:STM32L010K4T6
- added IC2: TMUX136RSER, Personal_Project:TMUX136RSER, symbol Personal_Projects:TMUX136RSER
- added J3: Data_Conn, Connector_PinHeader_2.54mm:PinHeader_1x04_P2.54mm_Horizontal, symbol Connector_Generic:Conn_01x04
- added J4: SEL Jumper, Connector_PinHeader_2.54mm:PinHeader_1x03_P2.54mm_Vertical, symbol Connector_Generic:Conn_01x03
- added J5: SW_Header, Connector_PinSocket_2.54mm:PinSocket_1x05_P2.54mm_Horizontal, symbol Connector_Generic:Conn_01x05
- added J6: BOOT Jumper, Connector_PinHeader_2.54mm:PinHeader_1x03_P2.54mm_Vertical, symbol Connector_Generic:Conn_01x03
- added U10, U11, U12, U13, U14, U15, U16, U17, U18, U19, U20, U21, U9: ~, Personal_Project:Button_KMR231GLFS, symbol Personal_Projects:Button_KMR231GLFS
Connections:
- net +3.3V: now also C10.1, C11.1, C14.1, C9.1, IC1.1 (VDD_1), IC1.17 (VDD_2), IC1.5 (VDDA), IC2.10 (VCC), J3.1 (Pin_1), J4.1 (Pin_1), J5.1 (Pin_1), J6.1 (Pin_1)
- net GND: now also C10.2, C11.2, C12.2, C13.2, C14.2, C15.2, C16.2, C17.2, C18.2, C19.2, C20.2, C21.2, C22.2, C23.2, C24.2, C25.2, C9.2, IC1.16 (VSS_1), IC1.2 (PC14-OSC32_IN), IC1.32 (VSS_2), IC2.5 (GND), IC2.6 (~{EN}), J3.2 (Pin_2), J4.3 (Pin_3), J5.2 (Pin_2), J6.3 (Pin_3), U10.3, U10.4, U10.5 (GND), U11.3, U11.4, U11.5 (GND), U12.3, U12.4, U12.5 (GND), U13.3, U13.4, U13.5 (GND), U14.3, U14.4, U14.5 (GND), U15.3, U15.4, U15.5 (GND), U16.3, U16.4, U16.5 (GND), U17.3, U17.4, U17.5 (GND), U18.3, U18.4, U18.5 (GND), U19.3, U19.4, U19.5 (GND), U20.3, U20.4, U20.5 (GND), U21.3, U21.4, U21.5 (GND), U9.3, U9.4, U9.5 (GND)
- new net BOOT0: IC1.31 (PB9-BOOT0), J6.2 (Pin_2)
- new net COM1: IC2.8 (COM1), J3.3 (Pin_3)
- new net COM2: IC2.7 (COM2), J3.4 (Pin_4)
- new net I2C1_SCL: IC1.29 (PB6), IC2.4 (B2)
- new net I2C1_SDA: IC1.30 (PB7), IC2.3 (B1)
- new net LPUART1_RX: IC1.6 (PA0-CK_IN), IC2.2 (A2)
- new net LPUART1_TX: IC1.7 (PA1), IC2.1 (A1)
- new net NRST: C12.1, IC1.4 (NRST), J5.5 (Pin_5), U9.1, U9.2
- new net PA10: C24.1, IC1.20 (PA10), U20.1, U20.2
- new net PA11: C25.1, IC1.21 (PA11), U21.1, U21.2
- new net PA2: C13.1, IC1.8 (PA2), U10.1, U10.2
- new net PA3: C15.1, IC1.9 (PA3), U11.1, U11.2
- new net PA4: C16.1, IC1.10 (PA4), U12.1, U12.2
- new net PA5: C17.1, IC1.11 (PA5), U13.1, U13.2
- new net PA6: C18.1, IC1.12 (PA6), U14.1, U14.2
- new net PA7: C19.1, IC1.13 (PA7), U15.1, U15.2
- new net PA8: C22.1, IC1.18 (PA8), U18.1, U18.2
- new net PA9: C23.1, IC1.19 (PA9), U19.1, U19.2
- new net PB0: C20.1, IC1.14 (PB0), U16.1, U16.2
- new net PB1: C21.1, IC1.15 (PB1), U17.1, U17.2
- new net SEL: IC2.9 (SEL), J4.2 (Pin_2)
- new net SYS_SWCLK: IC1.24 (PA14), J5.4 (Pin_4)
- new net SYS_SWDIO: IC1.23 (PA13), J5.3 (Pin_3)
- no-connect marks 0 -> 6
Other:
- note added: "If you won't use RTC or a 32 kHz clock: Tie OSC32_IN to GND Leave OSC32_OUT floating"
- note added: "SEL Switch select (logic Low = COM to A PORT Logic High = COM to B PORT) EN Enable (active low) The TMUX136 has internal 6-MΩ pull-down resistors on SEL and EN, so no external resistors are required on the logic pins. The internal pull-down resistor on SEL allows the PORT A channel to be selected by default. The internal pull-down resistor on EN enables the switch when power is applied to VCC."
- note removed: "1. Constructed with pull down resistors and own voltage to optional used on MCUs without own internal pull-up resistors. 2. 3V3 pins included in connector for so that the current doesnt generate signal in ther signal traces 3. Pin headers included for optional general connection 4. ESD protection included for potential elcrtrostatic discharge caused by pushing the buttons 5. Possibly add jupers t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"
- moved on the sheet: H1, H2, H3, H4

Commit message: update
Connections:
- net NRST: now also J5.3 (Pin_3); no longer J5.5 (Pin_5)
- net SYS_SWCLK: now also J5.5 (Pin_5); no longer J5.4 (Pin_4)
- net SYS_SWDIO: now also J5.4 (Pin_4); no longer J5.3 (Pin_3)
Other:
- note added: "If you won't use RTC or a 32 kHz clock: Tie OSC32_IN to GND Leave OSC32_OUT floating BOOT0 Cofiguration 1 MCU enters built-in bootloader mode, allowing firmware updates via UART or I2C. Used for flashing firmware without a debugger. 0 MCU starts normally, running the user program stored in internal flash. ✅ (Normal operation)"
- note removed: "If you won't use RTC or a 32 kHz clock: Tie OSC32_IN to GND Leave OSC32_OUT floating"
Changed lines of the file:
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@@
 		)
 	)
-	(text "If you won't use RTC or a 32 kHz clock:\n\nTie OSC32_IN to GND\nLeave OSC32_OUT floating\n"
+	(text "If you won't use RTC or a 32 kHz clock:\n\nTie OSC32_IN to GND\nLeave OSC32_OUT floating\n\nBOOT0 Cofiguration\n1 MCU enters built-in bootloader mode, allowing firmware \nupdates via UART or I2C. Used for flashing firmware \nwithout a debugger.\n0 MCU starts normally, running the user program stored \nin internal flash. ✅ (Normal operation)"
 		(exclude_from_sim no)
 		(at 330.2 46.355 0)
@@
 		)
 	)
+	(label "SYS_SWDIO"
+		(at 288.29 175.26 0)
+		(fields_autoplaced yes)
+		(effects
+			(font
+				(size 1.27 1.27)
+			)
+			(justify left bottom)
+		)
+	)
 	(label "I2C1_SCL"
 		(at 130.81 46.99 90)
@@
 		)
 	)
-	(label "NRST"
-		(at 288.29 177.8 0)
-		(fields_autoplaced yes)
-		(effects
-			(font
-				(size 1.27 1.27)
-			)
-			(justify left bottom)
-		)
-	)
 	(label "SEL"
 		(at 256.54 69.85 0)
@@
 		)
 	)
-	(label "SYS_SWCLK"
-		(at 288.29 175.26 0)
-		(fields_autoplaced yes)
-		(effects
-			(font
-				(size 1.27 1.27)
-			)
-			(justify left bottom)
-		)
-	)
 	(label "PA5"
 		(at 128.27 114.3 270)
@@
 		)
 	)
-	(label "SYS_SWDIO"
-		(at 288.29 172.72 0)
-		(fields_autoplaced yes)
-		(effects
-			(font
-				(size 1.27 1.27)
-			)
-			(justify left bottom)
-		)
-	)
 	(label "PA11"
 		(at 162.56 80.01 0)
@@
 		)
 	)
+	(label "SYS_SWCLK"
+		(at 288.29 177.8 0)
+		(fields_autoplaced yes)
+		(effects
+			(font
+				(size 1.27 1.27)
+			)
+			(justify left bottom)
+		)
+	)
 	(label "PA10"
 		(at 162.56 82.55 0)
@@
 		(fields_autoplaced yes)
 		(effects
+			(font
+				(size 1.27 1.27)
+			)
+			(justify left bottom)
+		)
+	)
+	(label "NRST"
+		(at 288.29 172.72 0)
+		(fields_autoplaced yes)
+		(effects

Commit message: Update
Other:
- company: (none) -> Peter Hancak
- title: (none) -> Keypad Board
Changed lines of the file:
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@@
 	(generator_version "8.0")
 	(paper "A3")
+	(title_block
+		(title "Keypad Board")
+		(date "2025-03-13")
+		(rev "A")
+		(company "Peter Hancak")
+	)
 	(junction
 		(at 227.33 208.28)

Commit message: Update
Connections:
- net NRST: now also J5.5 (Pin_5); no longer J5.3 (Pin_3)
- net SYS_SWCLK: now also J5.4 (Pin_4); no longer J5.5 (Pin_5)
- net SYS_SWDIO: now also J5.3 (Pin_3); no longer J5.4 (Pin_4)
Changed lines of the file:
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@@
-		)
-	)
-	(label "SYS_SWDIO"
-		(at 288.29 175.26 0)
-		(fields_autoplaced yes)
-		(effects
-			(font
-				(size 1.27 1.27)
-			)
-			(justify left bottom)
 		)
 	)
@@
 		)
 	)
+	(label "SYS_SWCLK"
+		(at 288.29 175.26 0)
+		(fields_autoplaced yes)
+		(effects
+			(font
+				(size 1.27 1.27)
+			)
+			(justify left bottom)
+		)
+	)
 	(label "PB0"
 		(at 50.8 207.01 90)
@@
 		)
 	)
+	(label "SYS_SWDIO"
+		(at 288.29 172.72 0)
+		(fields_autoplaced yes)
+		(effects
+			(font
+				(size 1.27 1.27)
+			)
+			(justify left bottom)
+		)
+	)
+	(label "NRST"
+		(at 288.29 177.8 0)
+		(fields_autoplaced yes)
+		(effects
+			(font
+				(size 1.27 1.27)
+			)
+			(justify left bottom)
+		)
+	)
 	(label "PB1"
 		(at 86.36 207.01 90)
@@
 		)
 	)
-	(label "SYS_SWCLK"
-		(at 288.29 177.8 0)
-		(fields_autoplaced yes)
-		(effects
-			(font
-				(size 1.27 1.27)
-			)
-			(justify left bottom)
-		)
-	)
 	(label "PA10"
 		(at 162.56 82.55 0)
@@
 		(fields_autoplaced yes)
 		(effects
-			(font
-				(size 1.27 1.27)
-			)
-			(justify left bottom)
-		)
-	)
-	(label "NRST"
-		(at 288.29 172.72 0)
-		(fields_autoplaced yes)
-		(effects

Commit message: Update
Connections:
- net SEL: now also IC1.25 (PA15)
- no-connect marks 6 -> 5
Changed lines of the file:
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@@
-	)
-	(no_connect
-		(at 140.97 54.61)
 	)
 	(no_connect
@@
 		(pts
 			(xy 50.8 182.88) (xy 50.8 184.15)
+		)
+		(stroke
+			(width 0)
+			(type default)
+		)
+	)
+	(wire
+		(pts
+			(xy 140.97 38.1) (xy 140.97 54.61)
 		)
 		(stroke
@@
 		(fields_autoplaced yes)
 		(effects
+			(font
+				(size 1.27 1.27)
+			)
+			(justify left bottom)
+		)
+	)
+	(label "SEL"
+		(at 140.97 41.91 90)
+		(fields_autoplaced yes)
+		(effects

Commit message: Update
Other:
- note added: "If you won't use RTC or a 32 kHz clock: Tie OSC32_IN to GND Leave OSC32_OUT floating BOOT0 Cofiguration 1 MCU enters built-in bootloader mode, allowing firmware updates via UART or I2C. Used for flashing firmware without a debugger. 0 MCU starts normally, running the user program stored in internal flash. ✅ (Normal operation) SEL Switch select (logic Low = COM to A PORT Logic High = COM to B PORT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"
- note removed: "If you won't use RTC or a 32 kHz clock: Tie OSC32_IN to GND Leave OSC32_OUT floating BOOT0 Cofiguration 1 MCU enters built-in bootloader mode, allowing firmware updates via UART or I2C. Used for flashing firmware without a debugger. 0 MCU starts normally, running the user program stored in internal flash. ✅ (Normal operation)"
Changed lines of the file:
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@@
 		)
 	)
-	(text "If you won't use RTC or a 32 kHz clock:\n\nTie OSC32_IN to GND\nLeave OSC32_OUT floating\n\nBOOT0 Cofiguration\n1 MCU enters built-in bootloader mode, allowing firmware \nupdates via UART or I2C. Used for flashing firmware \nwithout a debugger.\n0 MCU starts normally, running the user program stored \nin internal flash. ✅ (Normal operation)"
+	(text "If you won't use RTC or a 32 kHz clock:\nTie OSC32_IN to GND\nLeave OSC32_OUT floating\n\nBOOT0 Cofiguration\n1 MCU enters built-in bootloader mode, allowing firmware \nupdates via UART or I2C. Used for flashing firmware \nwithout a debugger.\n0 MCU starts normally, running the user program stored \nin internal flash. ✅ (Normal operation)\n\nSEL Switch select (logic Low = COM to A PORT Logic \nHigh = COM to B PORT) EN Enable (active low)\n\nThe TMUX136 has internal 6-MΩ pull-down resistors on \nSEL and EN, so no external resistors are required on \nthe logic pins. \nThe internal pull-down resistor on SEL allows the \nPORT A channel to be selected by default. The internal \npull-down resistor on EN enables the switch when power \nis applied to VCC."
 		(exclude_from_sim no)
-		(at 330.2 46.355 0)
+		(at 328.422 58.42 0)
 		(effects
 			(font
@@
 	(text "STM32MP157FAD1 2x\nSTM32WB55CGU6 2x\nSTM32WB5MMGH6TR\nSTM32MP135DAF7\nSTM32H7S7L8H6H\n\nSTSPIN958TR\nSTM32H7S3I8T6\nLSM6DSV16XTR\nISM330BXTR\nSTM32WL55CCU6\nSTM32WL55JCI6 2x"
 		(exclude_from_sim no)
-		(at 0.762 32.512 0)
+		(at -24.384 32.512 0)
 		(effects
 			(font

Commit message: Update
Parts:
- added J1: Data_Conn_Header, Connector_PinHeader_2.54mm:PinHeader_1x04_P2.54mm_Vertical, symbol Connector_Generic:Conn_01x04
- added J2: Pin_Header, Connector_PinHeader_2.54mm:PinHeader_1x04_P2.54mm_Vertical, symbol Connector_Generic:Conn_01x04
- added R1, R2, R3, R4: 100R, Resistor_SMD:R_0805_2012Metric_Pad1.20x1.40mm_HandSolder, symbol Device:R
- C10, C11, C12, C13, C14, C15, C16, C17, C18, C19, C20, C21, C22, C23, C24, C25, C9: footprint Capacitor_SMD:C_0805_2012Metric_Pad1.18x1.45mm_HandSolder -> Capacitor_SMD:C_0603_1608Metric_Pad1.08x0.95mm_HandSolder
- J3: value Data_Conn -> Data_Conn_Socket; footprint Connector_PinHeader_2.54mm:PinHeader_1x04_P2.54mm_Horizontal -> Connector_PinSocket_2.54mm:PinSocket_1x04_P2.54mm_Vertical
- J5: footprint Connector_PinSocket_2.54mm:PinSocket_1x05_P2.54mm_Horizontal -> Connector_PinHeader_2.54mm:PinHeader_1x05_P2.54mm_Vertical
Connections:
- net +3.3V: now also J1.1 (Pin_1)
- net COM1: now also J1.3 (Pin_3)
- net COM2: now also J1.4 (Pin_4)
- net GND: now also J1.2 (Pin_2)
- net I2C1_SCL: now also R4.1; no longer IC2.4 (B2)
- net I2C1_SDA: now also R3.1; no longer IC2.3 (B1)
- net LPUART1_RX: now also R2.1; no longer IC2.2 (A2)
- net LPUART1_TX: now also R1.1; no longer IC2.1 (A1)
- net PA12: now reaches IC1.22 (PA12)
- net PA12: now also J2.4 (Pin_4)
- net PB3: now reaches IC1.26 (PB3)
- net PB3: now also J2.3 (Pin_3)
- net PB4: now reaches IC1.27 (PB4)
- net PB4: now also J2.2 (Pin_2)
- net PB5: now reaches IC1.28 (PB5)
- net PB5: now also J2.1 (Pin_1)
- new net: IC2.1 (A1), R1.2
- new net: IC2.2 (A2), R2.2
- new net: IC2.3 (B1), R3.2
- new net: IC2.4 (B2), R4.2
- no-connect marks 5 -> 1
Other:
- moved on the sheet: C14, IC2, J3, J4

Commit message: Update
Connections:
- net PB3: now also J2.2 (Pin_2); no longer J2.3 (Pin_3)
- net PB4: now also J2.1 (Pin_1); no longer J2.2 (Pin_2)
- net SEL: now also IC1.28 (PB5); no longer IC1.25 (PA15)
- removed net PB5: IC1.28 (PB5), J2.1 (Pin_1)
- new net PA15: IC1.25 (PA15), J2.3 (Pin_3)
Changed lines of the file:
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@@
+		)
+	)
+	(label "PA15"
+		(at 140.97 43.18 90)
+		(effects
+			(font
+				(size 1.27 1.27)
+			)
+			(justify left bottom)
 		)
 	)
@@
 	(label "PB4"
 		(at 135.89 41.91 90)
+		(fields_autoplaced yes)
 		(effects
 			(font
@@
 		)
 	)
+	(label "SEL"
+		(at 133.35 38.1 270)
+		(fields_autoplaced yes)
+		(effects
+			(font
+				(size 1.27 1.27)
+			)
+			(justify right bottom)
+		)
+	)
 	(label "SYS_SWDIO"
 		(at 157.48 74.93 0)
@@
 	(label "PB3"
 		(at 138.43 41.91 90)
+		(fields_autoplaced yes)
 		(effects
 			(font
@@
 		)
 	)
+	(label "PB4"
+		(at 290.83 209.55 0)
+		(fields_autoplaced yes)
+		(effects
+			(font
+				(size 1.27 1.27)
+			)
+			(justify left bottom)
+		)
+	)
 	(label "PA3"
 		(at 86.36 163.83 90)
@@
 		)
 	)
-	(label "SEL"
-		(at 140.97 41.91 90)
-		(fields_autoplaced yes)
-		(effects
-			(font
-				(size 1.27 1.27)
-			)
-			(justify left bottom)
-		)
-	)
 	(label "PA5"
 		(at 128.27 114.3 270)
@@
 		)
 	)
+	(label "PA15"
+		(at 290.83 214.63 0)
+		(fields_autoplaced yes)
+		(effects
+			(font
+				(size 1.27 1.27)
+			)
+			(justify left bottom)
+		)
+	)
 	(label "BOOT0"
 		(at 95.25 45.72 0)
@@
 	(label "PA12"
 		(at 162.56 77.47 0)
-		(effects
-			(font
-				(size 1.27 1.27)
-			)
-			(justify left bottom)
-		)
-	)
-	(label "PB3"
-		(at 290.83 214.63 0)
 		(fields_autoplaced yes)
 		(effects
@@
 		)
 	)
-	(label "PB4"
-		(at 290.83 212.09 0)
-		(fields_autoplaced yes)
-		(effects
-			(font
-				(size 1.27 1.27)
-			)
-			(justify left bottom)
-		)
-	)
 	(label "PA12"
 		(at 290.83 217.17 0)
@@
 		)
 	)
-	(label "PB5"
-		(at 133.35 41.91 90)
-		(effects
-			(font
-				(size 1.27 1.27)
-			)
-			(justify left bottom)
-		)
-	)
 	(label "PA10"
 		(at 162.56 82.55 0)
@@
 		)
 	)
-	(label "PB5"
-		(at 290.83 209.55 0)
-		(fields_autoplaced yes)
-		(effects
+	(label "PB3"
+		(at 290.83 212.09 0)
+		(fields_autoplaced yes)
+		(effects
