File: Keypad_Board.kicad_sch (KiCad schematic)
At the start: 46 parts, among them IC1 STM32L010K4T6, IC2 TMUX136RSER, J1 Data_Conn_Header, J2 Pin_Header, J3 Data_Conn_Socket, J4 SEL Jumper, J5 SW_Header, J6 BOOT Jumper

Commit message: Update
Parts:
- added FB1: BLM21PG601SN1D_0805, Capacitor_SMD:C_0805_2012Metric_Pad1.18x1.45mm_HandSolder, symbol Device:FerriteBead
Connections:
- net +3.3V: now also FB1.1; no longer C11.1, IC1.5 (VDDA)
- new net VDDA: C11.1, FB1.2, IC1.5 (VDDA)
Other:
- moved on the sheet: C11, C12, U9

Commit message: Update
Parts:
- removed FB1: BLM21PG601SN1D_0805, Capacitor_SMD:C_0805_2012Metric_Pad1.18x1.45mm_HandSolder, symbol Device:FerriteBead
Connections:
- net VDDA is gone; now on net +3.3V: C11.1, IC1.5 (VDDA)
Changed lines of the file:
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@@
 	(wire
 		(pts
-			(xy 74.93 82.55) (xy 78.74 82.55)
+			(xy 83.82 82.55) (xy 91.44 82.55)
 		)
 		(stroke
@@
 	(wire
 		(pts
-			(xy 86.36 82.55) (xy 91.44 82.55)
-		)
-		(stroke
-			(width 0)
-			(type default)
-		)
-	)
-	(wire
-		(pts
 			(xy 96.52 176.53) (xy 96.52 179.07)
 		)
@@
 	(label "VDDA"
 		(at 106.68 82.55 180)
+		(fields_autoplaced yes)
 		(effects
 			(font
@@
 	)
 	(symbol
-		(lib_id "Device:FerriteBead")
-		(at 82.55 82.55 90)
-		(unit 1)
-		(exclude_from_sim no)
-		(in_bom yes)
-		(on_board yes)
-		(dnp no)
-		(property "Reference" "FB1"
-			(at 86.868 81.28 90)
-			(effects
-				(font
-					(size 1.27 1.27)
-				)
-			)
-		)
-		(property "Value" "BLM21PG601SN1D_0805"
-			(at 82.55 97.536 90)
-			(effects
-				(font
-					(size 1.27 1.27)
-				)
-			)
-		)
-		(property "Footprint" "Capacitor_SMD:C_0805_2012Metric_Pad1.18x1.45mm_HandSolder"
-			(at 82.55 84.328 90)
-			(effects
-				(font
-					(size 1.27 1.27)
-				)
-				(hide yes)
-			)
-		)
-		(property "Datasheet" "~"
-			(at 82.55 82.55 0)
-			(effects
-				(font
-					(size 1.27 1.27)
-				)
-				(hide yes)
-			)
-		)
-		(property "Description" "Ferrite bead"
-			(at 82.55 82.55 0)
-			(effects
-				(font
-					(size 1.27 1.27)
-				)
-				(hide yes)
-			)
-		)
-		(pin "1"
-		)
-		(pin "2"
-		)
-		(instances
-			(project "Keypad_Board"
-				(path "/4727cf53-8c99-4615-a2e8-49206f192bc9"
-					(reference "FB1")
-					(unit 1)
-				)
-			)
-		)
-	)
-	(symbol
 		(lib_id "power:GND")
 		(at 96.52 179.07 0)
@@
 	(symbol
 		(lib_id "power:+3.3V")
-		(at 74.93 82.55 90)
+		(at 83.82 82.55 90)
 		(unit 1)
 		(exclude_from_sim no)
@@
 		(dnp no)
 		(property "Reference" "#PWR047"
-			(at 78.74 82.55 0)
+			(at 87.63 82.55 0)
 			(effects
 				(font
@@
 		)
 		(property "Value" "+3.3V"
-			(at 72.39 84.074 90)
+			(at 81.28 84.074 90)
 			(effects
 				(font
@@
 		)
 		(property "Footprint" ""
-			(at 74.93 82.55 0)
+			(at 83.82 82.55 0)
 			(effects
 				(font
@@
 		)
 		(property "Datasheet" ""
-			(at 74.93 82.55 0)
+			(at 83.82 82.55 0)
 			(effects
 				(font
@@
 		)
 		(property "Description" "Power symbol creates a global label with name \"+3.3V\""
-			(at 74.93 82.55 0)
+			(at 83.82 82.55 0)
 			(effects
 				(font

Commit message: Update
Parts:
- removed R3, R4: 100R, Resistor_SMD:R_0805_2012Metric_Pad1.20x1.40mm_HandSolder, symbol Device:R
- R1, R2: value 100R -> 33R
Connections:
- net I2C1_SCL: now also IC2.4 (B2)
- net I2C1_SDA: now also IC2.3 (B1)
Changed lines of the file:
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@@
 	(wire
 		(pts
-			(xy 228.6 74.93) (xy 210.82 74.93)
+			(xy 210.82 74.93) (xy 241.3 74.93)
 		)
 		(stroke
@@
 	(wire
 		(pts
-			(xy 228.6 77.47) (xy 210.82 77.47)
+			(xy 210.82 77.47) (xy 241.3 77.47)
 		)
 		(stroke
@@
 	(wire
 		(pts
-			(xy 241.3 74.93) (xy 236.22 74.93)
-		)
-		(stroke
-			(width 0)
-			(type default)
-		)
-	)
-	(wire
-		(pts
 			(xy 151.13 77.47) (xy 167.64 77.47)
 		)
@@
 	(wire
 		(pts
-			(xy 241.3 77.47) (xy 236.22 77.47)
-		)
-		(stroke
-			(width 0)
-			(type default)
-		)
-	)
-	(wire
-		(pts
 			(xy 57.15 88.9) (xy 60.96 88.9)
 		)
@@
 			)
 		)
-		(property "Value" "100R"
+		(property "Value" "33R"
 			(at 237.744 68.834 90)
 			(effects
@@
 	(symbol
 		(lib_id "Device:R")
-		(at 232.41 77.47 90)
-		(unit 1)
-		(exclude_from_sim no)
-		(in_bom yes)
-		(on_board yes)
-		(dnp no)
-		(property "Reference" "R4"
-			(at 227.584 76.454 90)
-			(effects
-				(font
-					(size 1.27 1.27)
-				)
-			)
-		)
-		(property "Value" "100R"
-			(at 237.744 76.454 90)
-			(effects
-				(font
-					(size 1.27 1.27)
-				)
-			)
-		)
-		(property "Footprint" "Resistor_SMD:R_0805_2012Metric_Pad1.20x1.40mm_HandSolder"
-			(at 232.41 79.248 90)
-			(effects
-				(font
-					(size 1.27 1.27)
-				)
-				(hide yes)
-			)
-		)
-		(property "Datasheet" "~"
-			(at 232.41 77.47 0)
-			(effects
-				(font
-					(size 1.27 1.27)
-				)
-				(hide yes)
-			)
-		)
-		(property "Description" "Resistor"
-			(at 232.41 77.47 0)
-			(effects
-				(font
-					(size 1.27 1.27)
-				)
-				(hide yes)
-			)
-		)
-		(pin "1"
-		)
-		(pin "2"
-		)
-		(instances
-			(project "Keypad_Board"
-				(path "/4727cf53-8c99-4615-a2e8-49206f192bc9"
-					(reference "R4")
-					(unit 1)
-				)
-			)
-		)
-	)
-	(symbol
-		(lib_id "Device:R")
 		(at 232.41 72.39 90)
 		(unit 1)
@@
 			)
 		)
-		(property "Value" "100R"
+		(property "Value" "33R"
 			(at 237.744 71.374 90)
 			(effects
@@
 					(unit 1)
 				)
-			)
-		)
-	)
-	(symbol
-		(lib_id "Device:R")
-		(at 232.41 74.93 90)
-		(unit 1)
-		(exclude_from_sim no)
-		(in_bom yes)
-		(on_board yes)
-		(dnp no)
-		(property "Reference" "R3"
-			(at 227.584 73.914 90)
-			(effects
-				(font
-					(size 1.27 1.27)
-				)
-			)
-		)
-		(property "Value" "100R"
-			(at 237.744 73.914 90)
-			(effects
-				(font
-					(size 1.27 1.27)
-				)
-			)
-		)
-		(property "Footprint" "Resistor_SMD:R_0805_2012Metric_Pad1.20x1.40mm_HandSolder"
-			(at 232.41 76.708 90)
-			(effects
-				(font
-					(size 1.27 1.27)
-				)
-				(hide yes)
-			)
-		)
-		(property "Datasheet" "~"
-			(at 232.41 74.93 0)
-			(effects
-				(font
-					(size 1.27 1.27)
-				)
-				(hide yes)
-			)
-		)
-		(property "Description" "Resistor"
-			(at 232.41 74.93 0)
-			(effects
-				(font
-					(size 1.27 1.27)
-				)
-				(hide yes)
-			)
-		)
-		(pin "1"
-		)
-		(pin "2"
-		)
-		(instances
-			(project "Keypad_Board"
-				(path "/4727cf53-8c99-4615-a2e8-49206f192bc9"
-					(reference "R3")
-					(unit 1)
-				)

Commit message: Update
Other:
- note removed: "If you won't use RTC or a 32 kHz clock: Tie OSC32_IN to GND Leave OSC32_OUT floating BOOT0 Cofiguration 1 MCU enters built-in bootloader mode, allowing firmware updates via UART or I2C. Used for flashing firmware without a debugger. 0 MCU starts normally, running the user program stored in internal flash. ✅ (Normal operation) SEL Switch select (logic Low = COM to A PORT Logic High = COM to B PORT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"
Changed lines of the file:
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@@
 		)
 	)
-	(text_box "Notes"
+	(text_box "Notes:\n\nIf you won't use RTC or a 32 kHz clock:\nTie OSC32_IN to GND\nLeave OSC32_OUT floating\n\nBOOT0 Cofiguration\n1 MCU enters built-in bootloader mode, allowing firmware \nupdates via UART or I2C. Used for flashing firmware \nwithout a debugger.\n0 MCU starts normally, running the user program stored \nin internal flash. ✅ (Normal operation)\n\nSEL Switch select (logic Low = COM to A PORT Logic \nHigh = COM to B PORT) EN Enable (active low)\n\nThe TMUX136 has internal 6-MΩ pull-down resistors on \nSEL and EN, so no external resistors are required on \nthe logic pins. \nThe internal pull-down resistor on SEL allows the \nPORT A channel to be selected by default. The internal \npull-down resistor on EN enables the switch when power \nis applied to VCC.\n\nIncluded vertical pin header for I2C continuation"
 		(exclude_from_sim no)
 		(at 320.929 26.162 0)
@@
 		)
 	)
-	(text "If you won't use RTC or a 32 kHz clock:\nTie OSC32_IN to GND\nLeave OSC32_OUT floating\n\nBOOT0 Cofiguration\n1 MCU enters built-in bootloader mode, allowing firmware \nupdates via UART or I2C. Used for flashing firmware \nwithout a debugger.\n0 MCU starts normally, running the user program stored \nin internal flash. ✅ (Normal operation)\n\nSEL Switch select (logic Low = COM to A PORT Logic \nHigh = COM to B PORT) EN Enable (active low)\n\nThe TMUX136 has internal 6-MΩ pull-down resistors on \nSEL and EN, so no external resistors are required on \nthe logic pins. \nThe internal pull-down resistor on SEL allows the \nPORT A channel to be selected by default. The internal \npull-down resistor on EN enables the switch when power \nis applied to VCC.\n\nIncluded vertical pin header for I2C continuation"
-		(exclude_from_sim no)
-		(at 328.422 58.42 0)
-		(effects
-			(font
-				(size 1.27 1.27)
-			)
-			(justify left)
-		)
-	)
